Commit message: depth camera

File: description/depth_camera.xacro (robot description, xacro)
@@ -1,95 +1,90 @@
 <?xml version="1.0"?>
 <robot xmlns:xacro="http://www.ros.org/wiki/xacro">
-    <!-- <xacro:include filename="$(find realsense_ros2_gazebo)/xacro/depthcam.xacro"/> -->
-    <!-- <xacro:realsense_d435 sensor_name="d435" parent_link="base_link" rate="10"> -->
-    <!--     <origin rpy="0 0 0 " xyz="0 0 0.5"/> -->
-    <!-- </xacro:realsense_d435> -->
-    <joint name="camera_joint" type="fixed">
-        <parent link="chassis"/>
-        <child link="camera_link"/>
-        <origin xyz="0.306 0 0.16" rpy="0 0 0"/>
-    </joint>
-    <link name="camera_link">
-        <visual>
-            <geometry>
-                <box size="0.010 0.06 0.04"/>
-            </geometry>
-            <material name="orange"/>
-        </visual>
-    </link>
-    <link name="camera_rgb_optical_frame">
-        <inertial>
-            <pose>0.069 -0.047 0.107 0 0 0</pose>
-            <inertia>
-                <ixx>0.001</ixx>
-                <ixy>0.000</ixy>
-                <ixz>0.000</ixz>
-                <iyy>0.001</iyy>
-                <iyz>0.000</iyz>
-                <izz>0.001</izz>
-            </inertia>
-            <mass>0.035</mass>
-        </inertial>
-        <pose>0.069 -0.047 0.107 0 0 0</pose>
-        <sensor name="camera" type="depth">
-            <always_on>true</always_on>
-            <visualize>true</visualize>
-            <update_rate>30</update_rate>
-            <camera name="intel_realsense_d455">
-                <horizontal_fov>1.02974</horizontal_fov>
-                <image>
-                    <width>640</width>
-                    <height>480</height>
-                    <format>R8G8B8</format>
-                </image>
-                <clip>
-                    <near>0.02</near>
-                    <far>300</far>
-                </clip>
-                <noise>
-                    <type>gaussian</type>
-                    <!-- Noise is sampled independently per pixel on each frame.
-                  That pixel's noise value is added to each of its color
-                  channels, which at that point lie in the range [0,1]. -->
-                    <mean>0.0</mean>
-                    <stddev>0.007</stddev>
-                </noise>
-            </camera>
-            <plugin name="camera_driver" filename="libgazebo_ros_camera.so">
-                <ros>
-                    <!-- <namespace>test_cam</namespace> -->
-                    <!-- <remapping>image_raw:=image_demo</remapping> -->
-                    <!-- <remapping>camera_info:=camera_info_demo</remapping> -->
-                </ros>
-                <!-- camera_name>omit so it defaults to sensor name</camera_name-->
-                <!-- frame_name>omit so it defaults to link name</frameName-->
-                <!-- <hack_baseline>0.07</hack_baseline> -->
-            </plugin>
-        </sensor>
-    </link>
-    <link name="camera_rgb_frame" />
-    <joint name="camera_rgb_optical_joint" type="fixed">
-        <parent>camera_rgb_frame</parent>
-        <child>camera_rgb_optical_frame</child>
-        <pose>0 0 0 -1.57079632679 0 -1.57079632679</pose>
-        <axis>
-            <xyz>0 0 1</xyz>
-        </axis>
-    </joint>
-    <joint name="camera_joint" type="fixed">
-        <parent>base_link</parent>
-        <child>camera_link</child>
-        <pose>0.064 -0.065 0.094 0 0 0</pose>
-        <axis>
-            <xyz>0 0 1</xyz>
-        </axis>
-    </joint>
-    <joint name="camera_rgb_joint" type="fixed">
-        <parent>camera_link</parent>
-        <child>camera_rgb_frame</child>
-        <pose>0.005 0.018 0.013 0 0 0</pose>
-        <axis>
-            <xyz>0 0 1</xyz>
-        </axis>
-    </joint>
+  <joint name="camera_joint" type="fixed">
+    <parent link="chassis"/>
+    <child  link="camera_link"/>
+    <!-- <origin xyz="0.064 -0.065 0.094" rpy="0 0 0"/> -->
+    <origin xyz="0.307 0 0.16" rpy="0 0 0"/>
+  </joint>
+  <link name="camera_link">
+    <visual>
+      <geometry>
+        <box size="0.010 0.06 0.04"/>
+      </geometry>
+      <material name="orange"/>
+    </visual>
+  </link>
+  <!-- intermediate frame -->
+  <!-- <link name="camera_rgb_frame"/> -->
+  <!---->
+  <!-- <joint name="camera_rgb_joint" type="fixed"> -->
+  <!--   <parent link="camera_link"/> -->
+  <!--   <child  link="camera_rgb_frame"/> -->
+  <!-- <origin xyz="0.005 0.018 0.013" rpy="0 0 0"/> -->
+  <!--   <origin xyz="0 0 0" rpy="0 0 0"/> -->
+  <!-- </joint> -->
+  <!---->
+  <!-- optical frame with inertial expressed in URDF form -->
+  <link name="camera_rgb_optical_frame">
+    <inertial>
+      <!-- <origin xyz="0.069 -0.047 0.107" rpy="0 0 0"/> -->
+      <origin xyz="0 0 0" rpy="0 0 0"/>
+      <mass value="0.035"/>
+      <inertia ixx="0.001" ixy="0.0" ixz="0.0"
+               iyy="0.001" iyz="0.0" izz="0.001"/>
+    </inertial>
+  </link>
+  <joint name="camera_rgb_optical_joint" type="fixed">
+    <!-- <parent link="camera_rgb_frame"/> -->
+    <parent link="camera_link"/>
+    <child  link="camera_rgb_optical_frame"/>
+    <!-- rpy as in your original (roll, pitch, yaw) -->
+    <!-- <origin xyz="0 0 0" rpy="-1.57079632679 0 -1.57079632679"/> -->
+    <origin xyz="0 0 0" rpy="${-pi/2} 0 ${-pi/2}"/>
+    <!-- <origin xyz="0 0 0" rpy="0 0 0"/> -->
+  </joint>
+  <!-- <gazebo reference="camera_rgb_optical_frame"> -->
+  <gazebo reference="camera_link">
+    <sensor name="camera" type="depth">
+      <always_on>true</always_on>
+      <visualize>true</visualize>
+      <update_rate>30</update_rate>
+      <camera name="intel_realsense_d455">
+        <horizontal_fov>1.02974</horizontal_fov>
+        <image>
+          <width>640</width>
+          <height>480</height>
+          <format>B8G8R8</format>
+        </image>
+        <clip>
+          <!-- <near>0.02</near> -->
+          <!-- <far>300</far> -->
+          <near>0.02</near>
+          <far>20.0</far>
+        </clip>
+        <noise>
+          <type>gaussian</type>
+          <mean>0.0</mean>
+          <stddev>0.007</stddev>
+        </noise>
+      </camera>
+      <plugin name="camera_driver" filename="libgazebo_ros_camera.so">
+        <ros>
+          <namespace></namespace>
+        </ros>
+        <!-- Topics / frame -->
+        <camera_name>camera</camera_name>
+        <image_topic_name>image_raw</image_topic_name>
+        <camera_info_topic_name>camera_info</camera_info_topic_name>
+        <point_cloud_topic_name>points</point_cloud_topic_name>
+        <frame_name>camera_rgb_optical_frame</frame_name>
+        <!-- useful plugin params you can tune -->
+        <update_rate>30</update_rate>
+        <always_on>true</always_on>
+        <visualize>true</visualize>
+        <min_depth>0.1</min_depth>
+        <max_depth>100</max_depth>
+      </plugin>
+    </sensor>
+  </gazebo>
 </robot>

File: description/robot_core.xacro (robot description, xacro)
@@ -123,6 +123,6 @@
     <gazebo reference="caster_wheel">
         <material>Gazebo/Black</material>
-        <mu1 value="0.001"/>
-        <mu2 value="0.001"/>
+        <mu1 value="0.0001"/>
+        <mu2 value="0.0001"/>
     </gazebo>
 </robot>

Commit message: rtabmap rgbd. added imu to urdf

File: description/depth_camera.xacro (robot description, xacro)
@@ -24,14 +24,13 @@
   <!--   <origin xyz="0 0 0" rpy="0 0 0"/> -->
   <!-- </joint> -->
-  <!---->
   <!-- optical frame with inertial expressed in URDF form -->
   <link name="camera_rgb_optical_frame">
-    <inertial>
+    <!-- <inertial> -->
       <!-- <origin xyz="0.069 -0.047 0.107" rpy="0 0 0"/> -->
-      <origin xyz="0 0 0" rpy="0 0 0"/>
-      <mass value="0.035"/>
-      <inertia ixx="0.001" ixy="0.0" ixz="0.0"
-               iyy="0.001" iyz="0.0" izz="0.001"/>
-    </inertial>
+      <!-- <origin xyz="0 0 0" rpy="0 0 0"/> -->
+      <!-- <mass value="0.035"/> -->
+    <!--   <inertia ixx="0.001" ixy="0.0" ixz="0.0" -->
+    <!--            iyy="0.001" iyz="0.0" izz="0.001"/> -->
+    <!-- </inertial> -->
   </link>
   <joint name="camera_rgb_optical_joint" type="fixed">
@@ -61,5 +60,5 @@
           <!-- <far>300</far> -->
           <near>0.02</near>
-          <far>20.0</far>
+          <far>300</far>
         </clip>
         <noise>
@@ -70,7 +69,5 @@
       </camera>
       <plugin name="camera_driver" filename="libgazebo_ros_camera.so">
-        <ros>
-          <namespace></namespace>
-        </ros>
+        <ros></ros>
         <!-- Topics / frame -->
         <camera_name>camera</camera_name>
@@ -83,6 +80,6 @@
         <always_on>true</always_on>
         <visualize>true</visualize>
-        <min_depth>0.1</min_depth>
-        <max_depth>100</max_depth>
+        <min_depth>0.02</min_depth>
+        <max_depth>200</max_depth>
       </plugin>
     </sensor>

File: description/gazebo_control.xacro (robot description, xacro)
@@ -3,4 +3,5 @@
     <gazebo>
         <plugin name="diff_drive" filename="libgazebo_ros_diff_drive.so">
+            <update_rate>30.0</update_rate>
             <!-- Wheel Information -->
             <left_joint>left_wheel_joint</left_joint>
@@ -9,8 +10,9 @@
             <wheel_diameter>0.1</wheel_diameter>
             <!-- Limits -->
-            <max_wheel_torque>200</max_wheel_torque>
-            <max_wheel_acceleration>10.0</max_wheel_acceleration>
+            <max_wheel_torque>20</max_wheel_torque>
+            <max_wheel_acceleration>1.0</max_wheel_acceleration>
             <!-- Output -->
             <odometry_frame>odom</odometry_frame>
+            <odometry_topic>odom</odometry_topic>
             <robot_base_frame>base_link</robot_base_frame>
             <publish_odom>true</publish_odom>

File: description/robot.urdf.xacro (robot description, xacro)
@@ -1,8 +1,14 @@
 <?xml version="1.0"?>
 <robot xmlns:xacro="http://www.ros.org/wiki/xacro" name="robot">
+    <xacro:arg name="ros2_control" default="True"/>
     <xacro:include filename="robot_core.xacro"/>
-    <xacro:include filename="ros2_control.xacro"/>
-    <!-- <xacro:include filename="gazebo_control.xacro"/> -->
-    <xacro:include filename="lidar.xacro"/>
+    <xacro:if value="$(arg ros2_control)">
+        <xacro:include filename="ros2_control.xacro"/>
+    </xacro:if>
+    <xacro:unless value="$(arg ros2_control)">
+        <xacro:include filename="gazebo_control.xacro"/>
+    </xacro:unless>
+    <xacro:include filename="imu.xacro"/>
+    <!-- <xacro:include filename="lidar.xacro"/> -->
     <!-- <xacro:include filename="camera.xacro"/> -->
     <xacro:include filename="depth_camera.xacro"/>

File: description/robot_core.xacro (robot description, xacro)
@@ -18,6 +18,12 @@
     </material>
     <!-- BASE LINK -->
-    <link name="base_link">
-    </link>
+    <link name="base_link" />
+    <!-- BASE FOOTPRINT LINK-->
+    <joint name="base_footprint_joint" type="fixed">
+        <parent link="base_link"/>
+        <child link="base_footprint"/>
+        <origin xyz="0 0 0" rpy="0 0 0"/>
+    </joint>
+    <link name="base_footprint" />
     <!-- CHASSIS LINK -->
     <joint name="chassis_joint" type="fixed">
