Commit message: Changes for pick and place

File: software/ros_packages/rover_arm/config/rover_arm.ros2_control.xacro (robot description, xacro)
@@ -7,5 +7,5 @@
               <xacro:if value="${ros2_control_hardware_type == 'main'}">
                 <plugin>odrive_ros2_control_plugin/ODriveHardwareInterface</plugin>
-                <param name="can">can1</param>
+                <param name="can">can0</param>
                 <!-- <plugin>mock_components/GenericSystem</plugin> -->
               </xacro:if>

File: software/ros_packages/rover_arm_urdf/urdf/rover_arm.urdf (robot description, URDF)
Before this commit: robot rover_arm, 8 links, 7 joints
Links:
- added link jaws_link
Joints:
- added joint gripper_jaws: type fixed, parent arm_gripper, child jaws_link, origin xyz=0 0 0.10 rpy=0 0 0
