Commit message: pre-comp (hopefully) stable release.

File: software/ros_packages/rover_arm/config/rover_arm.urdf.xacro (robot description, xacro)
@@ -7,8 +7,4 @@
     <!-- Import control_xacro -->
     <xacro:include filename="rover_arm.ros2_control.xacro" />
-    <!-- Import odrive_drivebase urdf file -->
-    <xacro:include filename="$(find rover2_control)/rover2_control/drive_dummy.urdf" />
-    <!-- Import odrive_drivebase -->
-    <xacro:include filename="$(find rover2_control)/rover2_control/odrive_drive_ros2_control.xacro" />
     <!--Import camera-->
     <!-- Include sensors and other links -->

File: software/ros_packages/rover_arm_urdf/urdf/rover_arm.urdf (robot description, URDF)
Before this commit: robot rover_arm, 7 links, 6 joints
Joints:
- joint wrist_roll_joint: limit effort=1000.0 velocity=6.0 -> effort=1000.0 velocity=60.0

Commit message: Changed world transform to rover

File: software/ros_packages/rover_arm/config/rover_arm.urdf.xacro (robot description, xacro)
@@ -17,5 +17,5 @@
     <xacro:include filename="$(find realsense2_description)/urdf/_d455.urdf.xacro"/>
     <xacro:sensor_d455 parent="base_link" name="d455" use_nominal_extrinsics="true">
-        <origin xyz="-0.2 0.1 0" rpy="0 0 1.5707963267948"/>
+        <origin xyz="0.1 -0.2 0" rpy="0 0 0"/>
     </xacro:sensor_d455>
     <xacro:rover_arm_ros2_control name="RealSystem" initial_positions_file="$(arg initial_positions_file)" ros2_control_hardware_type="$(arg ros2_control_hardware_type)"/>

File: software/ros_packages/rover_arm_urdf/urdf/rover_arm.urdf (robot description, URDF)
Before this commit: robot rover_arm, 9 links, 8 joints
Links:
- removed link rover_body
- added link rover_base_origin; collision mesh filename=package://rover_arm_urdf/urdf/stl_files/rover_body.stl scale=0.001 0.001 0.001; visual mesh filename=package://rover_arm_urdf/urdf/stl_files/rover_body.stl scale=0.001 0.001 0.001
Joints:
- joint base_joint: origin xyz=0 0.055 0.087245 rpy=0 0 0 -> xyz=0.055 0 0.087245 rpy=0 0 -1.5708
- joint rover_body_joint: child rover_body -> base_link; origin xyz=0 0.084615 -0.03175 rpy=0 0 3.1415926 -> xyz=0.175735 0 0.03175 rpy=0 0 0; parent base_link -> rover_base_origin

Commit message: fix d455 orientation

File: software/ros_packages/rover_arm/config/rover_arm.urdf.xacro (robot description, xacro)
@@ -17,5 +17,5 @@
     <xacro:include filename="$(find realsense2_description)/urdf/_d455.urdf.xacro"/>
     <xacro:sensor_d455 parent="base_link" name="d455" use_nominal_extrinsics="true">
-        <origin xyz="0.1 -0.2 0" rpy="0 0 0"/>
+        <origin xyz="0.03 -0.075 -0.01" rpy="3.1415926536 0 0"/>
     </xacro:sensor_d455>
     <xacro:rover_arm_ros2_control name="RealSystem" initial_positions_file="$(arg initial_positions_file)" ros2_control_hardware_type="$(arg ros2_control_hardware_type)"/>
