Commit message: Added rover_body to Collision detection

File: software/ros_packages/rover_arm_urdf/urdf/rover_arm.urdf (robot description, URDF)
Before this commit: robot rover_arm, 7 links, 6 joints
Links:
- added link rover_body; collision mesh filename=package://rover_arm_urdf/urdf/stl_files/rover_body.stl scale=0.001 0.001 0.001; visual mesh filename=package://rover_arm_urdf/urdf/stl_files/rover_body.stl scale=0.001 0.001 0.001
Joints:
- added joint rover_body_joint: type fixed, parent base_link, child rover_body, origin xyz=0 0.084615 -0.03175 rpy=0 0 3.1415926

Commit message: Added visual segmentation to pick pipeline

File: software/ros_packages/rover_arm_urdf/urdf/rover_arm.urdf (robot description, URDF)
Before this commit: robot rover_arm, 9 links, 8 joints
Links:
- link jaws_link: geometry visual cylinder length=0.01 radius=0.005
Joints:
- joint gripper_jaws: origin xyz=0 0 0.10 rpy=0 0 0 -> xyz=0 0 0.23 rpy=0 0 0
